File: Hardware/CAN-Interface/Interface.sch (EAGLE design)
At the start: 53 parts, among them J1 34912-8020, J2 34912-8020, J3 34912-8020, J4 632722110112, J5 OBDII-FEMALEFEMALE, Q1 6.5A/20V/35mΩ, Q2 5.8A/30V/35mΩ, Q3 6.5A/20V/35mΩ, Q4 5.8A/30V/35mΩ

Commit message: pcb
Parts:
- removed J3: 34912-8020, SamacSys_Parts:34912-8020
- added C1-4: MINI50-4, interceptor:MINI50-4
- added D11: (no value), adafruit:DIODESOD-323F
- added F10: FUSE_CHIP-1206(3216-METRIC), Circuit-Protection:FUSE_CHIP-1206(3216-METRIC)
- added R9: 10k, interceptor:R0402
Connections:
- new net N$26: D4.A, Q1.G, R9.2
- new net N$27: D11.A, F10.2
- new net N$28: C1-4.1, D11.C
- net 12V: no longer J3.2
- net 12VIGN: now also F10.1
- net CAN1H: now also C1-4.2
- net CAN1L: now also C1-4.3
- net GND: now also C1-4.4, R9.1; no longer D4.A, J3.1, J3.3, J3.4, Q1.G
Other:
- moved on the sheet: C1-1, C1-2, C1-3, D1, D2, D3, F1, F2, F3, R3, SJ1
