File: Hardware/CAN-Interface/Interface.brd (EAGLE design)
At the start: 160 x 100 mm, 53 parts, among them J1 34912-8020, J2 34912-8020, J3 34912-8020, J4 632722110112, J5 OBDII-FEMALEFEMALE, Q1 6.5A/20V/35mΩ, Q2 5.8A/30V/35mΩ, Q3 6.5A/20V/35mΩ, Q4 5.8A/30V/35mΩ

Commit message: pcb
Parts:
- removed J3: 34912-8020, SamacSys_Parts:0349128020
- added C1-4: MINI50-4, interceptor:MINI50
- added D11: (no value), adafruit:SOD-323F
- added F10: FUSE_CHIP-1206(3216-METRIC), Circuit-Protection:FUSC3215X82N
- added R9: 10k, interceptor:0402-R
- moved U$1 205.5 mm to (91.0, 85.8), turned to 180 degrees
- moved D6 188.8 mm to (68.1, 11.9), flipped to the bottom, turned to 90 degrees
- moved R8 187.8 mm to (59.9, 83.0), turned to 180 degrees
- moved Q2 177.6 mm to (82.6, 73.4), turned to 90 degrees
- moved C1-9 173.2 mm to (84.7, 66.8), turned to 270 degrees
- moved SJ3 172.0 mm to (91.3, 50.1), flipped to the bottom, turned to 270 degrees
- moved D5 171.6 mm to (52.9, 11.8), flipped to the bottom, turned to 90 degrees
- moved SJ2 169.6 mm to (73.0, 9.68), flipped to the bottom
- moved Q3 169.3 mm to (82.6, 78.2), turned to 270 degrees
- moved Q1 168.4 mm to (90.6, 78.2), turned to 270 degrees
- moved F7 163.6 mm to (93.5, 30.4), flipped to the bottom
- moved F9 156.2 mm to (93.7, 60.8), flipped to the bottom
- moved C1-8 155.3 mm to (84.7, 51.6), turned to 270 degrees
- moved R4 153.5 mm to (73.1, 12.7), flipped to the bottom, turned to 180 degrees
- moved F5 148.2 mm to (68.1, 7.05), flipped to the bottom, turned to 90 degrees
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Connections:
- new net N$26: D4.1, Q1.4, R9.2
- new net N$27: D11.A, F10.2
- new net N$28: C1-4.4, D11.C
- net 12V: no longer J3.2
- net 12VIGN: now also F10.1
- net CAN1H: now also C1-4.3
- net CAN1L: now also C1-4.2
- net GND: now also C1-4.1, R9.1; no longer D4.1, J3.1, J3.3, J3.4, Q1.4
Routing:
- net CAN1L: track 0.00 -> 187.2 mm, vias 0 -> 3
- net CAN2L: track 0.00 -> 176.9 mm, vias 0 -> 1
- net CAN3L: track 0.00 -> 170.0 mm, vias 0 -> 4
- net CAN1H: track 0.00 -> 163.6 mm, vias 0 -> 5
- net CAN2H: track 0.00 -> 161.5 mm, vias 0 -> 6
- net CAN3H: track 0.00 -> 157.0 mm, vias 0 -> 2
- net 12VIGN: track 0.00 -> 108.0 mm, vias 0 -> 22
- net 12V: track 0.00 -> 89.5 mm, vias 0 -> 14
- net CAN4H: track 0.00 -> 33.8 mm, vias 0 -> 1
- net CAN4L: track 0.00 -> 29.8 mm
- net N$12: track 0.00 -> 17.4 mm
- net N$10: track 0.00 -> 13.8 mm
- net N$15: track 0.00 -> 8.40 mm
- net N$26: track 0.00 -> 5.40 mm
- net N$24: track 0.00 -> 4.26 mm
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- added copper zone on layer 1, net 12V
- added copper zone on layer 16, net 12V
- added copper zone on layer 1, net 12VIGN
- added copper zone on layer 16, net 12VIGN
- added copper zone on layer 1, net GND
- added copper zone on layer 16, net GND
Other:
- board size 160 x 100 mm -> 99.6 x 99.8 mm
- board text added: "CAN1 STEERING BRAKES PEDAL"
- board text added: "CAN2 CONTROLS"
- board text added: "CAN3 RADARS"
- board text added: "CONSTANT 12V"
- board text added: "OBD-2 GREY PANDA"
- board text added: "OBD-C CAUTION! C2/BLACK PANDA!"
- board text added: "POWER IN"

Commit message: Update Interface.brd
Routing:
- net CAN3L: track 170.0 -> 173.2 mm
Other:
- board text added: "OBD-C CAUTION! C2/BP ONLY!"
- board text removed: "OBD-C CAUTION! C2/BLACK PANDA!"
Changed lines of the file:
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@@
 <layer number="43" name="vRestrict" color="2" fill="10" visible="yes" active="yes"/>
 <layer number="44" name="Drills" color="7" fill="1" visible="no" active="yes"/>
-<layer number="45" name="Holes" color="7" fill="1" visible="no" active="yes"/>
+<layer number="45" name="Holes" color="7" fill="1" visible="yes" active="yes"/>
 <layer number="46" name="Milling" color="3" fill="1" visible="no" active="yes"/>
 <layer number="47" name="Measures" color="7" fill="1" visible="no" active="yes"/>
@@
 <text x="43" y="78" size="2.1844" layer="25" rot="SR180">OBD-2
 GREY PANDA</text>
-<text x="70" y="97" size="1.9304" layer="25" rot="SR180">OBD-C
+<text x="70" y="98.6" size="1.9304" layer="25" rot="SR180">OBD-C
 CAUTION!
-C2/BLACK PANDA!</text>
+C2/BP ONLY!</text>
 <wire x1="46" y1="0" x2="46" y2="38" width="0.1524" layer="25"/>
 <wire x1="46" y1="38" x2="26" y2="38" width="0.1524" layer="25"/>
@@
 <wire x1="26" y1="71" x2="26" y2="38" width="0.1524" layer="25"/>
 <wire x1="26" y1="71" x2="45" y2="71" width="0.1524" layer="25"/>
-<wire x1="45" y1="71" x2="45" y2="81" width="0.1524" layer="25"/>
-<wire x1="45" y1="81" x2="45" y2="100" width="0.1524" layer="25"/>
-<wire x1="45" y1="81" x2="71" y2="81" width="0.1524" layer="25"/>
-<wire x1="71" y1="81" x2="71" y2="100" width="0.1524" layer="25"/>
-<wire x1="71" y1="81" x2="73" y2="81" width="0.1524" layer="25"/>
-<wire x1="73" y1="81" x2="73" y2="71" width="0.1524" layer="25"/>
+<wire x1="45" y1="71" x2="45.1" y2="79.3" width="0.1524" layer="25"/>
+<wire x1="45.1" y1="79.3" x2="45" y2="100" width="0.1524" layer="25"/>
+<wire x1="45.1" y1="79.3" x2="71.1" y2="79.3" width="0.1524" layer="25"/>
+<wire x1="71.1" y1="79.3" x2="71" y2="100" width="0.1524" layer="25"/>
+<wire x1="71.1" y1="79.3" x2="73" y2="79.3" width="0.1524" layer="25"/>
+<wire x1="73" y1="79.3" x2="73" y2="71" width="0.1524" layer="25"/>
+<hole x="53.4" y="81.2" drill="3"/>
+<hole x="53.4" y="94.9" drill="3"/>
+<hole x="91.1" y="22" drill="3"/>
+<hole x="2.8" y="97.1" drill="3"/>
+<hole x="50" y="50.7" drill="3"/>
 </plain>
 <attributes>
@@
 <vertex x="0" y="99.8"/>
 </polygon>
+<via x="8.3" y="58.4" extent="1-16" drill="0.35"/>
+<via x="9.3" y="58.4" extent="1-16" drill="0.35"/>
+<via x="10.3" y="58.4" extent="1-16" drill="0.35"/>
+<via x="11.3" y="58.4" extent="1-16" drill="0.35"/>
+<via x="12.3" y="58.4" extent="1-16" drill="0.35"/>
+<via x="13.3" y="58.4" extent="1-16" drill="0.35"/>
+<via x="14.3" y="58.4" extent="1-16" drill="0.35"/>
+<via x="15.3" y="58.4" extent="1-16" drill="0.35"/>
+<via x="16.3" y="58.4" extent="1-16" drill="0.35"/>
+<via x="17.3" y="58.4" extent="1-16" drill="0.35"/>
+<via x="18.3" y="58.4" extent="1-16" drill="0.35"/>
+<via x="7.3" y="58.4" extent="1-16" drill="0.35"/>
 </signal>
 <signal name="N$12">
@@
 <wire x1="85.4" y1="75.538025" x2="85.4" y2="76.285" width="1.016" layer="1"/>
 <wire x1="86.035" y1="74.903025" x2="85.4" y2="75.538025" width="1.016" layer="1"/>
-<wire x1="53.4545" y1="89.6" x2="54.4" y2="90.5455" width="0.254" layer="16"/>
-<wire x1="54.4" y1="90.5455" x2="54.4" y2="96.4" width="0.254" layer="16"/>
+<wire x1="53.4545" y1="89.6" x2="55.4" y2="91.5455" width="0.254" layer="16"/>
+<wire x1="55.4" y1="91.5455" x2="55.4" y2="96.4" width="0.254" layer="16"/>
 <wire x1="52.64" y1="89.57" x2="52.67" y2="89.6" width="0.254" layer="1"/>
 <wire x1="52.67" y1="89.6" x2="53.4545" y2="89.6" width="0.254" layer="1"/>
@@
 <wire x1="55.27678125" y1="89.8914" x2="55.96321875" y2="89.8914" width="0.2032" layer="1"/>
 <wire x1="55.96321875" y1="89.8914" x2="56.4486" y2="90.37678125" width="0.2032" layer="1"/>
-<wire x1="56.4486" y1="90.37678125" x2="56.4486" y2="91.06321875" width="0.2032" layer="1"/>
+<wire x1="56.4486" y1="90.37678125" x2="56.4486" y2="95.06321875" width="0.2032" layer="1"/>
 <wire x1="54.3" y1="90.07" x2="55.09818125" y2="90.07" width="0.2032" layer="1"/>
 <wire x1="55.09818125" y1="90.07" x2="55.27678125" y2="89.8914" width="0.2032" layer="1"/>
-<wire x1="56.4486" y1="91.06321875" x2="51.61181875" y2="95.9" width="0.2032" layer="1"/>
-<wire x1="51.61181875" y1="95.9" x2="23.1" y2="95.9" width="0.2032" layer="1"/>
+<wire x1="56.4486" y1="95.06321875" x2="55.755909375" y2="95.755909375" width="0.2032" layer="1"/>
+<wire x1="55.755909375" y1="95.755909375" x2="55.61181875" y2="95.9" width="0.2032" layer="1"/>
 <wire x1="23.1" y1="95.9" x2="21.285" y2="94.085" width="0.2032" layer="1"/>
 <wire x1="21.285" y1="94.085" x2="21.285" y2="93" width="0.2032" layer="1"/>
+<wire x1="55.755909375" y1="95.755909375" x2="55.132384375" y2="95.755909375" width="0.254" layer="1"/>
+<wire x1="55.132384375" y1="95.755909375" x2="54.15809375" y2="96.7302" width="0.254" layer="1"/>
+<wire x1="23.9302" y1="96.7302" x2="23.1" y2="95.9" width="0.254" layer="1"/>
+<wire x1="54.15809375" y1="96.7302" x2="23.9302" y2="96.7302" width="0.254" layer="1"/>
 </signal>
 <signal name="N$29">

Commit message: clearance and power
Routing:
- net 12V: track 89.9 -> 92.1 mm, vias 14 -> 16
Changed lines of the file:
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@@
 <wire x1="85.4" y1="75.538025" x2="85.4" y2="76.285" width="1.016" layer="1"/>
 <wire x1="86.035" y1="74.903025" x2="85.4" y2="75.538025" width="1.016" layer="1"/>
-<wire x1="53.4545" y1="89.6" x2="55.4" y2="91.5455" width="0.254" layer="16"/>
-<wire x1="55.4" y1="91.5455" x2="55.4" y2="96.4" width="0.254" layer="16"/>
 <wire x1="52.64" y1="89.57" x2="52.67" y2="89.6" width="0.254" layer="1"/>
 <wire x1="52.67" y1="89.6" x2="53.4545" y2="89.6" width="0.254" layer="1"/>
@@
 <wire x1="53.4545" y1="89.6" x2="53.4545" y2="87.1245" width="0.254" layer="1"/>
 <wire x1="53.4545" y1="87.1245" x2="53.4" y2="87.07" width="0.254" layer="1"/>
+<via x="53.4545" y="88.6" extent="1-16" drill="0.35"/>
+<via x="53.4545" y="87.6" extent="1-16" drill="0.35"/>
+<wire x1="53.4545" y1="87.6" x2="53.4545" y2="88.6" width="0.3048" layer="16"/>
+<wire x1="53.4545" y1="88.6" x2="53.4545" y2="89.6" width="0.3048" layer="16"/>
+<wire x1="53.4545" y1="89.6" x2="53.6449" y2="89.7904" width="0.508" layer="16"/>
+<wire x1="53.6449" y1="89.7904" x2="53.75250625" y2="89.7904" width="0.508" layer="16"/>
+<wire x1="55.4" y1="91.88734375" x2="55.4" y2="96.5" width="0.508" layer="16"/>
+<wire x1="54.639" y1="91.12634375" x2="55.4" y2="91.88734375" width="0.508" layer="16"/>
+<wire x1="53.75250625" y1="89.7904" x2="54.639" y2="90.67689375" width="0.508" layer="16"/>
+<wire x1="54.639" y1="90.67689375" x2="54.639" y2="91.12634375" width="0.508" layer="16"/>
 </signal>
 <signal name="N$15">
@@
 <wire x1="55.09818125" y1="90.07" x2="55.27678125" y2="89.8914" width="0.2032" layer="1"/>
 <wire x1="56.4486" y1="95.06321875" x2="55.755909375" y2="95.755909375" width="0.2032" layer="1"/>
-<wire x1="55.755909375" y1="95.755909375" x2="55.61181875" y2="95.9" width="0.2032" layer="1"/>
 <wire x1="23.1" y1="95.9" x2="21.285" y2="94.085" width="0.2032" layer="1"/>
 <wire x1="21.285" y1="94.085" x2="21.285" y2="93" width="0.2032" layer="1"/>

Commit message: final board prep for manufacture
Changed lines of the file:
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@@
 </polygon>
 <wire x1="18.42" y1="66.41" x2="4.31" y2="66.41" width="1.016" layer="1"/>
-<wire x1="4.31" y1="66.41" x2="4.3" y2="66.4" width="1.016" layer="1"/>
 <wire x1="18.42" y1="47.36" x2="17.505" y2="48.275" width="1.016" layer="1"/>
 <wire x1="17.505" y1="48.275" x2="12.316975" y2="48.275" width="1.016" layer="1"/>
