File: Hardware/Tesla-Yaw-Emulator/yaw.sch (EAGLE design)
At the start: 31 parts, among them U1 STM32-M-64-LQFP, U2 MIC5233-5.0YM5-TR, U3 MIC5233-3.3YM5-TR, U4 TJA1042HVSON, Y1 16MHz

Commit message: yaw commit
Parts:
- removed C1, C2: 2.2uF, comma.ai:C0603
- removed C13, C9: 100nF, comma.ai:C0603
- removed D1: BAS40, diode:BAS40
- removed R10, R9: 5.1k, comma.ai:R0402
- removed R16, R17: 22, comma.ai:R0402
- removed S2: MOMENTARY-SWITCH-SPST-SMD-6.0X3.5MM, SparkFun-Switches:MOMENTARY-SWITCH-SPST-SMD-6.0X3.5MM
- removed U$3: MICROFIT-6, interceptor:MICROFIT-6
- added J1, J2: (no value), SparkFun-Connectors:CONN_08"
- C3, C4: value 12pF -> 22p
- J3: device ROTR-Wireless:USB-C-BREAKOUT_SPARKFUN-CONNECTORS_USB_C16PIN -> SparkFun-Connectors:CONN_05
- U1: value STM32-M-64-LQFP -> STM32F042K6U6; device comma.ai:STM32-M-64-LQFP -> interceptor:STM32F042K6U6
Connections:
- removed net ADC: U$3.2, U1.PC0-ADC10
- removed net ENC1: U$3.4, U1.PA8-USART1CK/TIM1CH1/OTG_FS_SOF
- removed net ENC2: U$3.5, U1.PA9-USART1TX/TIM1CH2/OTG_FS_VBUS
- removed net IO1: U$3.6, U1.PA10-USART1RX/TIM1CH3/OTG_FS_ID
- removed net N$7: S2.2, U1.BOOT0
- removed net VCAP1: C2.2, U1.VCAP1/[VSS]
- removed net VCAP2: C1.1, U1.VCAP2/[VSS]
- new net N$12: J2.1, U1A.PB0
- new net N$13: J2.2, U1A.PB1
- new net N$14: J2.3, U1A.PB2
- new net N$15: J2.4, U1A.PB3
- new net N$16: J2.5, U1A.PB4
- new net N$17: J2.6, U1A.PB5
- new net N$18: J2.7, U1A.PB6
- new net N$19: J2.8, U1A.PB7
- new net NRST: J3.4, S1.1, U1A.NRST
- new net SWC: J3.3, U1A.PA14
- new net SWD: J3.2, U1A.PA13
- new net VCC: J3.1
- net 3V3: now also U1B.VDD, U1B.VDDA, U1B.VDDIO2; no longer C13.1, C9.1, S2.1, U$3.3, U1.VDD1, U1.VDD2, U1.VDD3, U1.VDD4, U1.VDDA
- net 5V: no longer D1.C
- net CAN1_EN: now also U1A.PA10; no longer U1.PB3/JTDO-TIM2CH2/TRACESWO/SPI1SCK
- net CAN1_RX: now also U1A.PA11; no longer U1.PB8-TIM4CH3-I2C1SCL/CAN1_RX
- net CAN1_TX: now also U1A.PA12; no longer U1.PB9-TIM4CH4-I2C1SDA/CAN1_TX
- net GND: now also J3.5, S1.2, U1B.EPAD; no longer C1.2, C13.2, C2.1, C9.2, J3.GND, J3.SHLD, R10.1, R9.1, S1.1, U$3.1, U1.PB2/BOOT1, U1.VSS1, U1.VSS2, U1.VSSA
- net LEDG: now also U1A.PA15; no longer U1.PB11/[VCAP]
- net N$1: now also U1A.PF1-OSC_OUT; no longer U1.PH0-OSC_IN
- net N$10: now also J1.7, U1A.PA1; no longer S1.2, U1.NRST
- net N$11: now also J1.8, U1A.PA0; no longer D1.A, J3.VBUS
- net N$2: now also J1.1, U1A.PA7; no longer R16.1, U1.PA11-USART1CTS/OTG_FS_DM
- net N$3: now also U1A.PF0-OSC_IN; no longer U1.PH1-OSC_OUT
- net N$4: now also J1.2, U1A.PA6; no longer R17.1, U1.PA12-USART1RTS/OTG_FS_DP
- net N$5: now also J1.3, U1A.PA5; no longer J3.D-, R16.2
- net N$6: now also J1.4, U1A.PA4; no longer J3.D+, R17.2
- net N$8: now also J1.5, U1A.PA3; no longer J3.CC1, R9.2
- net N$9: now also J1.6, U1A.PA2; no longer J3.CC2, R10.2
Other:
- moved on the sheet: C3, C4, S1, Y1

Commit message: boards
Parts:
- added D1: DIODEDB2W40100L, comma.ai:DIODEDB2W40100L
- added J4: (no value), SparkFun-Connectors:CONN_05
- added R1, R2, R3, R4: (no value), comma.ai:R0402
- added S2: MOMENTARY-SWITCH-SPST-SMD-6.0X3.5MM, SparkFun-Switches:MOMENTARY-SWITCH-SPST-SMD-6.0X3.5MM
- J3: device SparkFun-Connectors:CONN_05 -> ROTR-Wireless:USB-C-BREAKOUT_SPARKFUN-CONNECTORS_USB_C16PIN
Connections:
- removed net N$1: C3.1, U1A.PF1-OSC_OUT, Y1.1
- removed net SWC: J3.3, U1A.PA14
- removed net SWD: J3.2, U1A.PA13
- removed net VCC: J3.1
- new net N$20: D1.A, J3.VBUS
- new net N$22: J3.D+, R1.1
- new net N$23: J3.D-, R2.1
- new net N$24: J3.CC1, R3.1
- new net N$25: J3.CC2, R4.1
- new net N$27: C4.1, U1A.PF1-OSC_OUT, Y1.2
- new net N$7: S2.1, U1A.PF11-BOOT0
- net 3V3: now also J4.4, S2.2
- net 5V: now also D1.C, J4.2
- net CAN1_RX: now also R1.2
- net CAN1_TX: now also R2.2
- net GND: now also J3.GND, J3.SHLD, J4.1, J4.3, J4.5, R3.2, R4.2; no longer J3.5
- net N$3: now also C3.1, Y1.1; no longer C4.1, Y1.2
- net NRST: no longer J3.4
