File: Hardware/Tesla-Yaw-Emulator/yaw.brd (EAGLE design)
At the start: 32.7 x 28 mm, 31 parts, among them U1 STM32-M-64-LQFP, U2 MIC5233-5.0YM5-TR, U3 MIC5233-3.3YM5-TR, U4 TJA1042HVSON, Y1 16MHz

Commit message: yaw commit
Parts:
- removed C1, C2: 2.2uF, comma.ai:0603-C
- removed C13, C9: 100nF, comma.ai:0603-C
- removed D1: BAS40, diode:SOT23
- removed R10, R9: 5.1k, comma.ai:0402-R
- removed R16, R17: 22, comma.ai:0402-R
- removed S2: MOMENTARY-SWITCH-SPST-SMD-6.0X3.5MM, SparkFun-Switches:TACTILE_SWITCH_SMD_6.0X3.5MM
- removed U$3: MICROFIT-6, interceptor:MICROFIT-6
- added J1, J2: (no value), SparkFun-Connectors:1X08
- C3, C4: value 12pF -> 22p
- J3: device ROTR-Wireless:USB-C-BREAKOUT_SPARKFUN-CONNECTORS_USB-C-16P -> SparkFun-Connectors:1X05
- U1: value STM32-M-64-LQFP -> STM32F042K6U6; device comma.ai:LQFP64 -> interceptor:UFQFPN32-5X5MM
- moved LED1 29.0 mm to (-13.4, 36.0)
- moved R13 28.6 mm to (-14.1, 30.4)
- moved J3 27.9 mm to (-2.00, 38.0)
- moved S1 14.8 mm to (11.4, 39.8), turned to 0 degrees
- moved U1 1.59 mm to (10.0, 45.0)
- moved C6 0.48 mm to (19.2, 47.7), turned to 180 degrees
Connections:
- removed net ADC: U$3.2, U1.8
- removed net ENC1: U$3.4, U1.41
- removed net ENC2: U$3.5, U1.42
- removed net IO1: U$3.6, U1.43
- removed net N$7: S2.2, U1.60
- removed net VCAP1: C2.2, U1.31
- removed net VCAP2: C1.1, U1.47
- new net N$12: J2.1, U1.14
- new net N$13: J2.2, U1.15
- new net N$14: J2.3, U1.16
- new net N$15: J2.4, U1.26
- new net N$16: J2.5, U1.27
- new net N$17: J2.6, U1.28
- new net N$18: J2.7, U1.29
- new net N$19: J2.8, U1.30
- new net NRST: J3.4, S1.1, U1.4
- new net SWC: J3.3, U1.24
- new net SWD: J3.2, U1.23
- new net VCC: J3.1
- net 3V3: now also U1.1, U1.17, U1.5; no longer C13.1, C9.1, S2.1, U$3.3, U1.13, U1.19, U1.32, U1.48, U1.64
- net 5V: no longer D1.3
- net CAN1_EN: now also U1.20; no longer U1.55
- net CAN1_RX: now also U1.21; no longer U1.61
- net CAN1_TX: now also U1.22; no longer U1.62
- net GND: now also J3.5, S1.2, U1.33; no longer C1.2, C13.2, C2.1, C9.2, J3.GND, J3.GND2, J3.SHLD1, J3.SHLD2, J3.SHLD3, J3.SHLD4, J3.SHLD5, J3.SHLD6, J3.SHLD7, J3.SHLD8, R10.1, R9.1, S1.1, U$3.1, U1.12, U1.18, U1.28, U1.63
- net LEDG: now also U1.25; no longer U1.30
- net N$1: now also U1.3; no longer U1.5
- net N$10: now also J1.7; no longer S1.2
- net N$11: now also J1.8, U1.6; no longer D1.1, J3.VBUS1, J3.VBUS2
- net N$2: now also J1.1, U1.13; no longer R16.1, U1.44
- net N$3: now also U1.2; no longer U1.6
- net N$4: now also J1.2, U1.12; no longer R17.1, U1.45
- net N$5: now also J1.3, U1.11; no longer J3.A7, J3.B7, R16.2
- net N$6: now also J1.4, U1.10; no longer J3.A6, J3.B6, R17.2
- net N$8: now also J1.5, U1.9; no longer J3.A5, R9.2
- net N$9: now also J1.6, U1.8; no longer J3.B5, R10.2
Routing:
- net 3V3: track 79.9 -> 26.3 mm, vias 7 -> 1
- net N$7: track 53.5 -> 0.00 mm, vias 2 -> 0
- net N$10: track 46.2 -> 0.00 mm, vias 2 -> 0
- net ADC: track 36.5 -> 0.00 mm, vias 1 -> 0
- net ENC1: track 25.0 -> 0.00 mm, vias 2 -> 0
- net ENC2: track 22.0 -> 0.00 mm, vias 2 -> 0
- net IO1: track 19.8 -> 0.00 mm, vias 2 -> 0
- net 5V: track 41.0 -> 22.2 mm, vias 2 -> 0
- net CAN1_EN: track 18.0 -> 1.03 mm, vias 3 -> 1
- net N$4: track 15.2 -> 0.00 mm
- net N$2: track 14.2 -> 0.00 mm
- net N$11: track 13.7 -> 0.00 mm, vias 1 -> 0
- net CAN1_TX: track 12.0 -> 0.00 mm, vias 1 -> 0
- net CAN1_RX: track 10.8 -> 0.00 mm, vias 1 -> 0
- net N$5: track 6.53 -> 0.00 mm
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Other:
- board size 32.7 x 28 mm -> 32.7 x 17 mm
- board text removed: "B"
- board text removed: "OUT"

Commit message: boards
Parts:
- added D1: DIODEDB2W40100L, comma.ai:SOD-123F
- added J4: (no value), SparkFun-Connectors:1X05
- added R1, R2, R3, R4: (no value), comma.ai:0402-R
- added S2: MOMENTARY-SWITCH-SPST-SMD-6.0X3.5MM, SparkFun-Switches:TACTILE_SWITCH_SMD_6.0X3.5MM
- J3: device SparkFun-Connectors:1X05 -> ROTR-Wireless:USB-C-BREAKOUT_SPARKFUN-CONNECTORS_USB-C-16P
- moved R13 32.4 mm to (13.5, 47.4), flipped to the bottom, turned to 180 degrees
- moved LED1 32.1 mm to (18.7, 36.4), turned to 180 degrees
- moved C11 9.46 mm to (19.0, 49.6), turned to 180 degrees
- moved J3 5.80 mm to (1.40, 42.7), turned to 270 degrees
- moved C10 5.52 mm to (11.0, 44.2), turned to 90 degrees
- moved J2 2.84 mm to (16.2, 49.5)
- moved J1 2.69 mm to (16.4, 35.3)
- moved C12 2.22 mm to (8.22, 42.6), turned to 180 degrees
- moved Y1 2.00 mm to (5.53, 44.1)
- moved C3 2.00 mm to (4.54, 45.9)
- moved C4 2.00 mm to (4.58, 39.9)
- moved C14 1.00 mm to (27.7, 38.2)
- moved C7 1.00 mm to (27.8, 44.5)
- moved U2 1.00 mm to (27.8, 47.6)
- moved U3 1.00 mm to (27.8, 41.3)
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Connections:
- removed net N$1: C3.1, U1.3, Y1.1
- removed net SWC: J3.3, U1.24
- removed net SWD: J3.2, U1.23
- removed net VCC: J3.1
- new net N$20: D1.2, J3.VBUS1, J3.VBUS2
- new net N$22: J3.A6, J3.B6, R1.1
- new net N$23: J3.A7, J3.B7, R2.1
- new net N$24: J3.A5, R3.1
- new net N$25: J3.B5, R4.1
- new net N$27: C4.1, U1.3, Y1.3
- new net N$7: S2.1, U1.31
- net 3V3: now also J4.4, S2.2
- net 5V: now also D1.1, J4.2
- net CAN1_RX: now also R1.2
- net CAN1_TX: now also R2.2
- net GND: now also J3.GND, J3.GND2, J3.SHLD1, J3.SHLD2, J3.SHLD3, J3.SHLD4, J3.SHLD5, J3.SHLD6, J3.SHLD7, J3.SHLD8, J4.1, J4.3, J4.5, R3.2, R4.2; no longer J3.5
- net N$3: now also C3.1, Y1.1; no longer C4.1, Y1.3
- net NRST: no longer J3.4
Routing:
- net 3V3: track 26.3 -> 60.8 mm, vias 1 -> 6
- net N$26: track 0.00 -> 29.3 mm, vias 0 -> 1
- net N$11: track 0.00 -> 15.1 mm, vias 0 -> 2
- net N$20: track 0.00 -> 15.0 mm, vias 0 -> 1
- net N$12: track 0.00 -> 13.2 mm, vias 0 -> 2
- net N$10: track 0.00 -> 12.9 mm, vias 0 -> 2
- net N$19: track 0.00 -> 12.1 mm
- net N$2: track 0.00 -> 10.9 mm
- net N$13: track 0.00 -> 10.9 mm, vias 0 -> 2
- net N$18: track 0.00 -> 10.5 mm
- net N$9: track 0.00 -> 10.4 mm, vias 0 -> 2
- net N$14: track 0.00 -> 10.2 mm, vias 0 -> 2
- net 5V: track 22.2 -> 32.1 mm, vias 0 -> 2
- net N$6: track 0.00 -> 9.59 mm
- net N$8: track 0.00 -> 9.01 mm
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Other:
- board size 32.7 x 17 mm -> 37.7 x 16.9 mm

Commit message: Update yaw.brd
Parts:
- moved R2 47.9 mm to (4.70, 44.9), turned to 90 degrees
- moved R4 46.1 mm to (-0.90, 41.0)
- moved R3 46.0 mm to (-0.70, 43.8)
- moved R1 41.1 mm to (2.50, 43.5), turned to 90 degrees
- moved R13 0.50 mm to (13.5, 47.9)
- moved C11 0.22 mm to (19.1, 49.8)
Routing:
- net CAN1_RX: track 4.91 -> 24.8 mm
- net N$7: track 0.00 -> 18.1 mm, vias 0 -> 2
- net CAN1_TX: track 5.75 -> 21.7 mm
- net N$23: track 2.67 -> 5.74 mm, vias 0 -> 1
- net GND: track 3.23 -> 6.14 mm, vias 4 -> 5
- net N$24: track 0.00 -> 2.83 mm, vias 0 -> 1
- net N$22: track 2.67 -> 5.18 mm, vias 0 -> 1
- net N$25: track 0.00 -> 2.50 mm, vias 0 -> 1
- net CAN1_EN: track 9.32 -> 11.4 mm

Commit message: signal switching
Routing:
- net 5V: track 32.1 -> 58.8 mm
Changed lines of the file:
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@@
 <wire x1="26.87" y1="44.4" x2="26.94" y2="44.47" width="0.508" layer="16"/>
 <wire x1="24.7344" y1="40.9025375" x2="23.5874625" y2="39.7556" width="0.3048" layer="16"/>
-<wire x1="18.06486875" y1="41.71" x2="17.81" y2="41.71" width="0.3048" layer="16"/>
+<wire x1="18.06486875" y1="41.71" x2="18" y2="41.71" width="0.3048" layer="16"/>
+<wire x1="18" y1="41.71" x2="17.81" y2="41.71" width="0.3048" layer="16"/>
 <wire x1="24.7344" y1="41.7644" x2="24.7344" y2="40.9025375" width="0.3048" layer="16"/>
 <wire x1="26.94" y1="44.47" x2="26.94" y2="43.97" width="0.3048" layer="16"/>
@@
 <wire x1="16.8" y1="42.8" x2="16.8" y2="42.72" width="0.254" layer="16"/>
 <wire x1="16.8" y1="42.72" x2="17.81" y2="41.71" width="0.254" layer="16"/>
-<wire x1="-3" y1="40.5" x2="16.415221875" y2="44.684778125" width="0" layer="19" extent="16-16"/>
+<wire x1="-3" y1="40.5" x2="-0.8444" y2="38.3444" width="0.3048" layer="16"/>
+<wire x1="-0.8444" y1="38.3444" x2="-0.8444" y2="38.0571625" width="0.3048" layer="16"/>
+<wire x1="-0.8444" y1="38.0571625" x2="0.2127625" y2="37" width="0.3048" layer="16"/>
+<wire x1="17" y1="37" x2="18" y2="38" width="0.3048" layer="16"/>
+<wire x1="18" y1="38" x2="18" y2="41.71" width="0.3048" layer="16"/>
+<wire x1="0.2127625" y1="37" x2="17" y2="37" width="0.3048" layer="16"/>
 </signal>
 <signal name="CAN1_RX">
