File: Hardware/Tesla-Translator-Emulator/trans-emu.brd (EAGLE design)
At the start: 160 x 100 mm, 33 parts, among them IC1 MIC5233-3.3YM5-TR, U1 STM32F413RGT6, U2 TJA1042HVSON, U3 TJA1042HVSON, U4 TJA1042HVSON, Y1 CRYSTAL-3.2X2.54-PIN

Commit message: boards
Parts:
- moved C5 82.2 mm to (25.8, 14.0), flipped to the bottom, turned to 90 degrees
- moved C4 71.2 mm to (17.9, 15.0), flipped to the bottom, turned to 90 degrees
- moved C3 67.0 mm to (19.7, 20.5), flipped to the bottom, turned to 270 degrees
- moved R3 64.7 mm to (22.1, 9.39), turned to 180 degrees
- moved C1 62.5 mm to (24.8, 26.6), turned to 270 degrees
- moved R4 61.8 mm to (15.5, 9.40)
- moved C13 61.5 mm to (15.3, 28.4), turned to 90 degrees
- moved C2 59.9 mm to (18.2, 26.6), turned to 90 degrees
- moved R2 59.8 mm to (17.6, 9.39), turned to 180 degrees
- moved R1 59.8 mm to (20.1, 9.39), turned to 180 degrees
- moved C16 58.8 mm to (12.4, 2.76), flipped to the bottom, turned to 90 degrees
- moved D1 56.6 mm to (11.1, 6.82), flipped to the bottom, turned to 270 degrees
- moved C8 55.7 mm to (23.1, 19.2), flipped to the bottom
- moved C14 55.1 mm to (4.73, 28.7), turned to 90 degrees
- moved C12 53.4 mm to (11.9, 32.1)
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Connections:
- net N$1: no longer C2.1
- net N$2: now also C2.1
Routing:
- net 3.3V: track 0.00 -> 104.2 mm, vias 0 -> 8
- net 5V: track 0.00 -> 79.5 mm, vias 0 -> 4
- net CAN3_EN: track 0.00 -> 36.6 mm, vias 0 -> 3
- net CAN1_EN: track 0.00 -> 35.0 mm, vias 0 -> 3
- net CAN2_EN: track 0.00 -> 33.2 mm, vias 0 -> 3
- net CAN2_TX: track 0.00 -> 32.3 mm, vias 0 -> 3
- net CAN2_RX: track 0.00 -> 30.4 mm, vias 0 -> 3
- net CAN3_TX: track 0.00 -> 25.2 mm, vias 0 -> 3
- net CAN1_TX: track 0.00 -> 22.4 mm, vias 0 -> 3
- net 12V: track 0.00 -> 20.7 mm
- net N$8: track 0.00 -> 20.4 mm, vias 0 -> 2
- net N$2: track 0.00 -> 19.8 mm
- net CAN1_RX: track 0.00 -> 18.9 mm, vias 0 -> 1
- net N$1: track 0.00 -> 18.5 mm
- net CAN3_RX: track 0.00 -> 16.4 mm, vias 0 -> 1
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- added copper zone on layer 1, net GND
- added copper zone on layer 16, net GND
Other:
- board size 160 x 100 mm -> 29 x 34 mm
- board text added: "B"
- board text added: "IN"
- board text added: "OUT"
- board text added: "Ocelot CAN Translator"
- board text added: "R"

Commit message: final board prep for manufacture
Parts:
- added R5, R6: 120, comma.ai:0402-R
Connections:
- net CAN2_H: now also R5.1
- net CAN2_L: now also R5.2
- net CAN3_H: now also R6.1
- net CAN3_L: now also R6.2
Routing:
- net CAN3_L: track 3.01 -> 4.44 mm
- net CAN2_H: track 8.99 -> 10.0 mm
- net GND: track 10.7 -> 9.74 mm, vias 7 -> 11
- net CAN2_L: track 11.1 -> 11.7 mm
Changed lines of the file:
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@@
 </element>
 <element name="C14" library="comma.ai" package="0603-C" value="100n" x="4.73298125" y="28.734240625" smashed="yes" rot="MR90">
-<attribute name="NAME" x="5.89498125" y="27.145240625" size="0.6096" layer="26" rot="MR90"/>
+<attribute name="NAME" x="5.57758125" y="26.3343625" size="0.6096" layer="26" rot="MR0"/>
 </element>
 <element name="C15" library="comma.ai" package="0603-C" value="2.2u" x="4.9647" y="5.02721875" smashed="yes" rot="MR180">
@@
 </element>
 <element name="C7" library="comma.ai" package="0603-C" value="100n" x="23.05558125" y="21.3334625" smashed="yes" rot="MR0">
-<attribute name="NAME" x="24.64458125" y="22.4954625" size="0.6096" layer="26" rot="MR0"/>
+<attribute name="NAME" x="25.4089375" y="21.147" size="0.6096" layer="26" rot="MR270"/>
 </element>
 <element name="C8" library="comma.ai" package="0603-C" value="100n" x="23.07081875" y="19.248121875" smashed="yes" rot="MR0">
-<attribute name="NAME" x="24.65981875" y="20.410121875" size="0.6096" layer="26" rot="MR0"/>
+<attribute name="NAME" x="25.327659375" y="19.061659375" size="0.6096" layer="26" rot="MR270"/>
 </element>
 <element name="C9" library="comma.ai" package="0603-C" value="100n" x="7.020878125" y="19.65268125" smashed="yes" rot="MR0">
@@
 </element>
 <element name="U3" library="comma.ai" package="HVSON8" value="TJA1042HVSON" x="1.9952625" y="28.77271875" smashed="yes" rot="MR270">
-<attribute name="NAME" x="0.1752625" y="30.39271875" size="0.254" layer="20" rot="MR270"/>
+<attribute name="NAME" x="0.469903125" y="26.92815625" size="0.254" layer="20" rot="MR270"/>
 </element>
 <element name="U4" library="comma.ai" package="HVSON8" value="TJA1042HVSON" x="12.09" y="28.52" smashed="yes" rot="MR270">
@@
 <element name="Y1" library="comma.ai" package="XTAL-3.2X2.5" value="CRYSTAL-3.2X2.54-PIN" x="20.372996875" y="27.58831875" smashed="yes">
 <attribute name="NAME" x="19.672996875" y="28.38831875" size="0.6096" layer="21"/>
+</element>
+<element name="R5" library="comma.ai" package="0402-R" value="120" x="8.700259375" y="23.498821875" smashed="yes" rot="MR180">
+<attribute name="NAME" x="8.065259375" y="22.736821875" size="0.6096" layer="26" rot="MR180"/>
+</element>
+<element name="R6" library="comma.ai" package="0402-R" value="120" x="8.9144" y="25.78278125" smashed="yes" rot="MR270">
+<attribute name="NAME" x="9.236978125" y="27.924" size="0.6096" layer="26" rot="MR270"/>
 </element>
 </elements>
@@
 </polygon>
 <wire x1="24.89" y1="11.63" x2="24.892540625" y2="11.627459375" width="0.254" layer="1"/>
-<wire x1="24.892540625" y1="11.627459375" x2="24.892540625" y2="10.6266625" width="0.254" layer="1"/>
 <via x="25.740921875" y="9.419221875" extent="1-16" drill="0.35"/>
 <wire x1="24.89" y1="11.63" x2="24.9836" y2="11.5364" width="0.254" layer="1"/>
@@
 <wire x1="17.00544375" y1="16.00290625" x2="17.00290625" y2="16.00290625" width="0.508" layer="16"/>
 <via x="17.00290625" y="16.00290625" extent="1-16" drill="0.3048"/>
-<wire x1="17.00290625" y1="16.00290625" x2="17" y2="16" width="0.508" layer="1"/>
-<wire x1="25.7937" y1="14.855559375" x2="24.89" y2="11.63" width="0" layer="19" extent="1-16"/>
+<via x="24.894540625" y="10.576559375" extent="1-16" drill="0.35"/>
+<via x="24" y="15" extent="1-16" drill="0.35"/>
+<via x="23.187659375" y="15.3035" extent="1-16" drill="0.35"/>
+<via x="25.847040625" y="10.614659375" extent="1-16" drill="0.35"/>
 </signal>
 <signal name="CAN1_RX">
@@
 <wire x1="7.32" y1="23.29130625" x2="7.32" y2="22.25" width="0.254" layer="16"/>
 <wire x1="5.935" y1="24.67630625" x2="7.32" y2="23.29130625" width="0.254" layer="16"/>
+<contactref element="R5" pad="1"/>
+<wire x1="8.250259375" y1="23.498821875" x2="8.04274375" y2="23.29130625" width="0.1524" layer="16"/>
+<wire x1="8.04274375" y1="23.29130625" x2="7.32" y2="23.29130625" width="0.1524" layer="16"/>
 </signal>
 <signal name="CAN2_L">
@@
 <wire x1="2.5162625" y1="26.79250625" x2="2.666709375" y2="26.642059375" width="0.254" layer="16"/>
 <wire x1="2.666709375" y1="26.642059375" x2="5.971540625" y2="26.642059375" width="0.254" layer="16"/>
-<wire x1="6.316" y1="24.834125" x2="6.904125" y2="24.246" width="0.254" layer="16"/>
+<wire x1="6.316" y1="24.834125" x2="6.942225" y2="24.2079" width="0.254" layer="16"/>
 <wire x1="5.971540625" y1="26.642059375" x2="6.316" y2="26.2976" width="0.254" layer="16"/>
-<wire x1="6.904125" y1="24.246" x2="7.755459375" y2="24.246" width="0.254" layer="16"/>
+<wire x1="6.942225" y1="24.2079" x2="8.829878125" y2="24.2079" width="0.254" layer="16"/>
 <wire x1="6.316" y1="26.2976" x2="6.316" y2="24.834125" width="0.254" layer="16"/>
-<wire x1="9.751459375" y1="22.25" x2="10.32" y2="22.25" width="0.254" layer="16"/>
-<wire x1="7.755459375" y1="24.246" x2="9.751459375" y2="22.25" width="0.254" layer="16"/>
+<wire x1="10.32" y1="22.25" x2="10.32" y2="22.717778125" width="0.254" layer="16"/>
+<wire x1="10.32" y1="22.717778125" x2="9.364978125" y2="23.6728" width="0.254" layer="16"/>
+<contactref element="R5" pad="2"/>
+<wire x1="9.364978125" y1="23.6728" x2="8.829878125" y2="24.2079" width="0.254" layer="16"/>
+<wire x1="9.150259375" y1="23.498821875" x2="9.3242375" y2="23.6728" width="0.1524" layer="16"/>
+<wire x1="9.3242375" y1="23.6728" x2="9.364978125" y2="23.6728" width="0.1524" layer="16"/>
 </signal>
 <signal name="CAN3_H">
@@
 <wire x1="11.569" y1="26.5397875" x2="11.308053125" y2="26.278840625" width="0.254" layer="16"/>
 <wire x1="8.348840625" y1="26.278840625" x2="7.32" y2="25.25" width="0.254" layer="16"/>
-<wire x1="11.308053125" y1="26.278840625" x2="8.348840625" y2="26.278840625" width="0.254" layer="16"/>
+<wire x1="11.308053125" y1="26.278840625" x2="9" y2="26.278840625" width="0.254" layer="16"/>
+<contactref element="R6" pad="1"/>
+<wire x1="9" y1="26.278840625" x2="8.348840625" y2="26.278840625" width="0.254" layer="16"/>
+<wire x1="8.9144" y1="26.23278125" x2="8.960459375" y2="26.278840625" width="0.1524" layer="16"/>
+<wire x1="8.960459375" y1="26.278840625" x2="9" y2="26.278840625" width="0.1524" layer="16"/>
 </signal>
 <signal name="CAN3_L">
@@
 <wire x1="12.219" y1="26.5397875" x2="10.9292125" y2="25.25" width="0.254" layer="16"/>
 <wire x1="10.9292125" y1="25.25" x2="10.32" y2="25.25" width="0.254" layer="16"/>
+<contactref element="R6" pad="2"/>
+<wire x1="10.32" y1="25.25" x2="8.99718125" y2="25.25" width="0.1524" layer="16"/>
+<wire x1="8.99718125" y1="25.25" x2="8.9144" y2="25.33278125" width="0.1524" layer="16"/>
 </signal>
 <signal name="N$2">

Commit message: signal switching
Parts:
- added Q1: PMOSFET, Transistor:SOT23
- added Q2: NMOSFET, Transistor:SOT23
- added R7, R8: 10k, comma.ai:0402-R
Connections:
- new net N$15: Q1.3, U$2.4
- new net N$16: Q1.1, Q2.3, R7.1
- new net PWRON: Q2.1, R8.2, U1.33
- net 12V: now also Q1.2, R7.2; no longer U$2.4
- net GND: now also Q2.2, R8.1
Routing:
- net PWRON: track 0.00 -> 18.6 mm, vias 0 -> 2
- net 12V: track 20.7 -> 15.0 mm
- net N$16: track 0.00 -> 4.94 mm, vias 0 -> 1
- net N$15: track 0.00 -> 4.36 mm
- net GND: track 9.74 -> 13.3 mm, vias 11 -> 12
- net 5V: track 79.5 -> 78.9 mm
