File: Hardware/Universal-Controls/control.sch (EAGLE design)
At the start: 44 parts, among them U1 STM32-M-64-LQFP, U2 MIC5233-5.0YM5-TR, U3 MIC5233-3.3YM5-TR, U4 TJA1042HVSON, U6 MCP6002, Y1 16MHz

Commit message: Button controller commit
Parts:
- removed C26: 100nF, comma.ai:C0603
- removed R1, R2, R3, R4, R7, R8: 10k, comma.ai:R0402
- removed R23, R24, R25, R26: 1k, comma.ai:R0402
- removed U$1: MICROFIT-6, interceptor:MICROFIT-6
- removed U6: MCP6002, comma.ai:LM358D
Connections:
- removed net ACCEL1: R23.2, U$3.2
- removed net ACCEL2: R24.2, U$3.5
- removed net DAC1: R3.2, U$1.2, U6A.OUT
- removed net DAC2: R2.2, U$1.5, U6B.OUT
- removed net DACV: C26.1, U$1.3, U$1.6, U6P.V+
- removed net N$17: R7.2, U1.PA4-SPI1NSS/ADC4/USART2CK/DAC_OUT1, U6A.+IN
- removed net N$18: R8.2, U1.PA5-SPI1SCK/ADC5/DAC_OUT2, U6B.+IN
- removed net N$21: R1.2, R3.1, U6A.-IN
- removed net N$22: R2.1, R4.2, U6B.-IN
- removed net N$41: R23.1, R26.1, U1.PC0-ADC10
- removed net N$42: R24.1, R25.1, U1.PC1-ADC11
- new net ADC: U$3.2, U1.PC0-ADC10
- new net ENC1: U$3.4, U1.PA8-USART1CK/TIM1CH1/OTG_FS_SOF
- new net ENC2: U$3.5, U1.PA9-USART1TX/TIM1CH2/OTG_FS_VBUS
- new net IO1: U$3.6, U1.PA10-USART1RX/TIM1CH3/OTG_FS_ID
- net 3V3: now also U$3.3
- net 5V: no longer U$3.3, U$3.6
- net GND: no longer C26.2, R1.1, R25.2, R26.2, R4.1, R7.1, R8.1, U$1.1, U$1.4, U$3.4, U6P.V-
Other:
- note removed: "*"
- note removed: "*0.1% precision"

Commit message: add pull resistors
Parts:
- added R1, R2: (no value), comma.ai:R0402
Connections:
- net 3V3: now also R2.1
- net GND: now also R1.1
- net N$10: now also R2.2
- net N$7: now also R1.2
Changed lines of the file:
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@@
 <setting verticaltext="up"/>
 </settings>
-<grid distance="0.1" unitdist="inch" unit="inch" style="dots" multiple="1" display="yes" altdistance="5" altunitdist="mil" altunit="mil"/>
+<grid distance="0.1" unitdist="inch" unit="inch" style="lines" multiple="1" display="no" altdistance="0.01" altunitdist="inch" altunit="inch"/>
 <layers>
 <layer number="1" name="Top" color="4" fill="1" visible="no" active="no"/>
@@
 <part name="U$3" library="interceptor" deviceset="MICROFIT-6" device=""/>
 <part name="SUPPLY8" library="SparkFun-Aesthetics" library_urn="urn:adsk.eagle:library:507" deviceset="VCC" device="" value="3V3"/>
+<part name="R1" library="comma.ai" deviceset="R" device="0402"/>
+<part name="R2" library="comma.ai" deviceset="R" device="0402"/>
+<part name="SUPPLY4" library="SparkFun-Aesthetics" library_urn="urn:adsk.eagle:library:507" deviceset="VCC" device="" value="3V3"/>
+<part name="GND7" library="SparkFun-Aesthetics" library_urn="urn:adsk.eagle:library:507" deviceset="GND" device=""/>
 </parts>
 <sheets>
@@
 <instance part="SUPPLY8" gate="G$1" x="148.59" y="81.534" smashed="yes">
 <attribute name="VALUE" x="147.574" y="85.09" size="1.778" layer="96"/>
+</instance>
+<instance part="R1" gate="G$1" x="190.5" y="149.86" smashed="yes" rot="R90">
+<attribute name="NAME" x="189.0014" y="146.05" size="1.778" layer="95" rot="R90"/>
+<attribute name="VALUE" x="193.802" y="146.05" size="1.778" layer="96" rot="R90"/>
+</instance>
+<instance part="R2" gate="G$1" x="71.12" y="160.02" smashed="yes" rot="R90">
+<attribute name="NAME" x="69.6214" y="156.21" size="1.778" layer="95" rot="R90"/>
+<attribute name="VALUE" x="74.422" y="156.21" size="1.778" layer="96" rot="R90"/>
+</instance>
+<instance part="SUPPLY4" gate="G$1" x="68.58" y="147.32" smashed="yes" rot="R180">
+<attribute name="VALUE" x="69.596" y="143.764" size="1.778" layer="96" rot="R180"/>
+</instance>
+<instance part="GND7" gate="1" x="190.5" y="142.24" smashed="yes">
+<attribute name="VALUE" x="187.96" y="139.7" size="1.778" layer="96"/>
 </instance>
 </instances>
@@
 <pinref part="C14" gate="G$1" pin="2"/>
 <pinref part="GND21" gate="1" pin="GND"/>
+</segment>
+<segment>
+<pinref part="R1" gate="G$1" pin="1"/>
+<pinref part="GND7" gate="1" pin="GND"/>
 </segment>
 </net>
@@
 <pinref part="U$3" gate="G$1" pin="3"/>
 </segment>
+<segment>
+<pinref part="R2" gate="G$1" pin="1"/>
+<pinref part="SUPPLY4" gate="G$1" pin="VCC"/>
+<wire x1="68.58" y1="147.32" x2="71.12" y2="154.94" width="0.1524" layer="91"/>
+<label x="66.04" y="152.4" size="1.778" layer="95"/>
+</segment>
 </net>
 <net name="N$1" class="0">
@@
 <pinref part="S1" gate="G$1" pin="2"/>
 <wire x1="73.66" y1="165.1" x2="71.12" y2="165.1" width="0.1524" layer="91"/>
+<pinref part="R2" gate="G$1" pin="2"/>
+<junction x="71.12" y="165.1"/>
 </segment>
 </net>
@@
 <pinref part="S2" gate="G$1" pin="2"/>
 <pinref part="U1" gate="G$1" pin="BOOT0"/>
-<wire x1="193.04" y1="157.48" x2="185.42" y2="157.48" width="0.1524" layer="91"/>
-</segment>
-</net>
+<wire x1="193.04" y1="157.48" x2="190.5" y2="157.48" width="0.1524" layer="91"/>
+<pinref part="R1" gate="G$1" pin="2"/>
+<wire x1="190.5" y1="157.48" x2="185.42" y2="157.48" width="0.1524" layer="91"/>
+<wire x1="190.5" y1="154.94" x2="190.5" y2="157.48" width="0.1524" layer="91"/>
+<junction x="190.5" y="157.48"/>
+</segment>
+</net>
