File: Hardware/STM32-Teensy/stm32teensy.sch (EAGLE design)
At the start: 24 parts, among them U1 STM32F413CGU3, U2 AP2112K-3.3TRG1, Y1 CRYSTAL-3.2X2.54-PIN

Commit message: Ibooster board updates
Parts:
- C5, C6: value (none) -> 22p
Changed lines of the file:
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@@
 <part name="C3" library="comma.ai" deviceset="C" device="0402" value="100n"/>
 <part name="C4" library="comma.ai" deviceset="C" device="0402" value="100n"/>
-<part name="C5" library="comma.ai" deviceset="C" device="0402"/>
-<part name="C6" library="comma.ai" deviceset="C" device="0402"/>
+<part name="C5" library="comma.ai" deviceset="C" device="0402" value="22p"/>
+<part name="C6" library="comma.ai" deviceset="C" device="0402" value="22p"/>
 <part name="Y1" library="comma.ai" deviceset="CRYSTAL-3.2X2.5" device="4-PIN"/>
 <part name="GND2" library="SparkFun-PowerSymbols" library_urn="urn:adsk.eagle:library:530" deviceset="GND" device=""/>
